File: elec/layout/default/stm32l432kbu6.kicad_pcb (KiCad board)
At the start: 2 copper layers, 225.7 x 100.8 mm, 0 parts

Commit message: intial layout
Parts:
- added C1: 10V 4.7uF X5R ±20% 0402 Multilayer Ceramic Capacitors MLCC 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, lib:C0402, F.Cu at (156.3, 111.5)
- added C2: 16V 100nF X7R ±10% 0402 Multilayer Ceramic Capacitors MLCC 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, lib:C0402, F.Cu at (164.7, 114.1)
- added C3: 25V 1uF X5R ±10% 0402 Multilayer Ceramic Capacitors MLCC - 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, lib:C0402, F.Cu at (156.3, 109.1)
- added C4: 16V 100nF X7R ±10% 0402 Multilayer Ceramic Capacitors MLCC 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, lib:C0402, F.Cu at (164.7, 113.0)
- added C5: 50V 10nF X7R ±10% 0402 Multilayer Ceramic Capacitors MLCC -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, lib:C0402, F.Cu at (156.3, 108.1)
- added C6: 50V 13pF C0G ±2% 0402 Multilayer Ceramic Capacitors MLCC - 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, lib:C0402, F.Cu at (157.9, 115.8)
- added C7: 50V 13pF C0G ±2% 0402 Multilayer Ceramic Capacitors MLCC - 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, lib:C0402, F.Cu at (156.3, 112.6)
- added R1: 62.5mW Thick Film Resistors ±100ppm/℃ ±1% 330Ω 0402 Chip Re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, lib:R0402, F.Cu at (160.5, 106.7)
- added R2: 62.5mW Thick Film Resistors ±100ppm/℃ ±1% 10kΩ 0402 Chip Re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, lib:R0402, F.Cu at (158.9, 106.7)
- added U1: , lib:UFQFPN-32_L5.0-W5.0-P0.50-TL-EP3.5, F.Cu at (160.6, 111.2)
- added U2: , lib:FC-135R_L3.2-W1.5, F.Cu at (156.1, 115.0)
Routing:
- net gnd: track 0.00 -> 20.6 mm, vias 0 -> 4
- net pc14_osc32_in: track 0.00 -> 12.5 mm
- net vcc: track 0.00 -> 8.88 mm, vias 0 -> 4
- net pc15_osc32_out: track 0.00 -> 8.52 mm
- net ph3_boot0: track 0.00 -> 1.62 mm
- net tx: track 0.00 -> 1.52 mm
