File: elec/layout/default/stm32l432kbu6.kicad_pcb (KiCad board)
At the start: 2 copper layers, 225.7 x 100.8 mm, 11 parts

Commit message: update layout
Connections:
- net vcc renamed ic-vcc
Changed lines of the file:
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@@
   (net 0 "")
   (net 1 "tx")
-  (net 2 "vcc")
+  (net 2 "ic-vcc")
   (net 3 "ph3_boot0")
   (net 4 "gnd")
@@
       (stroke (width 0.1) (type solid)) (layer "F.Fab"))
     (pad "1" smd roundrect (at -0.48 0) (size 0.56 0.62) (layers "F.Cu" "F.Paste" "F.Mask") (roundrect_rratio 0.25)
-      (net 2 "vcc") (pintype "stereo"))
+      (net 2 "ic-vcc") (pintype "stereo"))
     (pad "2" smd roundrect (at 0.48 0) (size 0.56 0.62) (layers "F.Cu" "F.Paste" "F.Mask") (roundrect_rratio 0.25)
       (net 4 "gnd") (pintype "stereo"))
@@
       (stroke (width 0.1) (type solid)) (layer "F.Fab"))
     (pad "1" smd roundrect (at -0.48 0 180) (size 0.56 0.62) (layers "F.Cu" "F.Paste" "F.Mask") (roundrect_rratio 0.25)
-      (net 2 "vcc") (pintype "stereo"))
+      (net 2 "ic-vcc") (pintype "stereo"))
     (pad "2" smd roundrect (at 0.48 0 180) (size 0.56 0.62) (layers "F.Cu" "F.Paste" "F.Mask") (roundrect_rratio 0.25)
       (net 4 "gnd") (pintype "stereo"))
@@
       (stroke (width 0.1) (type solid)) (layer "F.Fab"))
     (pad "1" smd roundrect (at -0.48 0) (size 0.56 0.62) (layers "F.Cu" "F.Paste" "F.Mask") (roundrect_rratio 0.25)
-      (net 2 "vcc") (pintype "stereo"))
+      (net 2 "ic-vcc") (pintype "stereo"))
     (pad "2" smd roundrect (at 0.48 0) (size 0.56 0.62) (layers "F.Cu" "F.Paste" "F.Mask") (roundrect_rratio 0.25)
       (net 4 "gnd") (pintype "stereo"))
@@
       (net 1 "tx") (pintype "stereo"))
     (pad "2" smd roundrect (at 0.51 0 90) (size 0.54 0.64) (layers "F.Cu" "F.Paste" "F.Mask") (roundrect_rratio 0.25)
-      (net 2 "vcc") (pintype "stereo"))
+      (net 2 "ic-vcc") (pintype "stereo"))
     (model "${KICAD6_3DMODEL_DIR}/Resistor_SMD.3dshapes/R_0402_1005Metric.wrl"
       (offset (xyz 0 0 0))
@@
       (stroke (width 0.1) (type solid)) (layer "F.Fab"))
     (pad "1" smd roundrect (at -0.48 0 180) (size 0.56 0.62) (layers "F.Cu" "F.Paste" "F.Mask") (roundrect_rratio 0.25)
-      (net 2 "vcc") (pintype "stereo"))
+      (net 2 "ic-vcc") (pintype "stereo"))
     (pad "2" smd roundrect (at 0.48 0 180) (size 0.56 0.62) (layers "F.Cu" "F.Paste" "F.Mask") (roundrect_rratio 0.25)
       (net 4 "gnd") (pintype "stereo"))
@@
       (stroke (width 0.1) (type solid)) (layer "F.Fab"))
     (pad "1" smd roundrect (at -0.48 0 180) (size 0.56 0.62) (layers "F.Cu" "F.Paste" "F.Mask") (roundrect_rratio 0.25)
-      (net 2 "vcc") (pintype "stereo"))
+      (net 2 "ic-vcc") (pintype "stereo"))
     (pad "2" smd roundrect (at 0.48 0 180) (size 0.56 0.62) (layers "F.Cu" "F.Paste" "F.Mask") (roundrect_rratio 0.25)
       (net 4 "gnd") (pintype "stereo"))
@@
       (stroke (width 0.06) (type solid)) (fill none) (layer "F.Fab"))
     (pad "1" smd rect (at -2.49 -1.75) (size 0.75 0.28) (layers "F.Cu" "F.Paste" "F.Mask")
-      (net 2 "vcc") (pintype "stereo"))
+      (net 2 "ic-vcc") (pintype "stereo"))
     (pad "2" smd rect (at -2.49 -1.25) (size 0.75 0.28) (layers "F.Cu" "F.Paste" "F.Mask")
       (net 5 "pc14_osc32_in") (pintype "stereo"))
@@
       (net 29 "nrst") (pintype "stereo"))
     (pad "5" smd rect (at -2.49 0.25) (size 0.75 0.28) (layers "F.Cu" "F.Paste" "F.Mask")
-      (net 2 "vcc") (pintype "stereo"))
+      (net 2 "ic-vcc") (pintype "stereo"))
     (pad "6" smd rect (at -2.49 0.75) (size 0.75 0.28) (layers "F.Cu" "F.Paste" "F.Mask")
       (net 28 "pa0_ck_in") (pintype "stereo"))
@@
       (net 4 "gnd") (pintype "stereo"))
     (pad "17" smd rect (at 2.49 1.75) (size 0.75 0.28) (layers "F.Cu" "F.Paste" "F.Mask")
-      (net 2 "vcc") (pintype "stereo"))
+      (net 2 "ic-vcc") (pintype "stereo"))
     (pad "18" smd rect (at 2.49 1.25) (size 0.75 0.28) (layers "F.Cu" "F.Paste" "F.Mask")
       (net 18 "pa8") (pintype "stereo"))
